File: HF_front.brd (EAGLE design)
At the start: 50 x 34 mm, 34 parts, among them U1 MC12080, U2 MAX9203, U3 HMC476MP86, U4 HMC476MP86

Commit message: more minor pcb changes
Parts:
- added R6: 50, resistor:R0603
Connections:
- net GND: now also R6.1
- net N$6: now also R6.2
Routing:
- net N$6: track 2.43 -> 3.93 mm
Changed lines of the file:
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@@
 <setting verticaltext="up"/>
 </settings>
-<grid distance="0.05" unitdist="inch" unit="inch" style="lines" multiple="1" display="yes" altdistance="0.00625" altunitdist="inch" altunit="inch"/>
+<grid distance="0.0125" unitdist="inch" unit="inch" style="lines" multiple="1" display="yes" altdistance="0.00625" altunitdist="inch" altunit="inch"/>
 <layers>
 <layer number="1" name="Top" color="4" fill="1" visible="yes" active="yes"/>
@@
 <text x="46.355" y="6.6675" size="1.524" layer="22" font="vector" rot="MR0">GND</text>
 <text x="46.355" y="12.065" size="1.524" layer="22" font="vector" rot="MR0">OUT</text>
+<rectangle x1="11.1125" y1="25.7175" x2="13.335" y2="27.305" layer="41"/>
+<rectangle x1="11.43" y1="20.955" x2="13.0175" y2="22.5425" layer="41"/>
+<rectangle x1="32.0675" y1="20.955" x2="34.6075" y2="22.5425" layer="41"/>
+<rectangle x1="32.0675" y1="24.765" x2="34.6075" y2="27.305" layer="41"/>
 </plain>
 <attributes>
@@
 <element name="C17" library="resistor" package="C0603" value="100n" x="42.2275" y="13.6525"/>
 <element name="JP1" library="pinhead" package="1X08" value="" x="48.26" y="16.51" rot="MR270"/>
+<element name="R6" library="resistor" package="R0603" value="50" x="36.83" y="21.9075" rot="R90"/>
 </elements>
 <signals>
@@
 <via x="34.6075" y="20.32" extent="1-16" drill="0.3" shape="octagon"/>
 <via x="35.56" y="20.32" extent="1-16" drill="0.3" shape="octagon"/>
-<via x="36.5125" y="20.32" extent="1-16" drill="0.3" shape="octagon"/>
+<via x="36.5125" y="20.0025" extent="1-16" drill="0.3" shape="octagon"/>
 <via x="18.7325" y="23.1775" extent="1-16" drill="0.3" shape="octagon"/>
 <via x="18.7325" y="24.13" extent="1-16" drill="0.3" shape="octagon"/>
@@
 <via x="43.4975" y="8.89" extent="1-16" drill="0.3" shape="octagon"/>
 <via x="42.545" y="8.89" extent="1-16" drill="0.3" shape="octagon"/>
+<contactref element="R6" pad="1"/>
 </signal>
 <signal name="+5V">
@@
 <contactref element="C2" pad="2"/>
 <contactref element="U1" pad="1"/>
-<wire x1="36.41" y1="24.13" x2="38.8366" y2="24.13" width="1.016" layer="1"/>
+<wire x1="36.41" y1="24.13" x2="37.1475" y2="24.13" width="1.016" layer="1"/>
+<contactref element="R6" pad="2"/>
+<wire x1="37.1475" y1="24.13" x2="38.8366" y2="24.13" width="1.016" layer="1"/>
+<wire x1="36.83" y1="22.7575" x2="36.83" y2="23.8125" width="0.8128" layer="1"/>
+<wire x1="36.83" y1="23.8125" x2="37.1475" y2="24.13" width="0.8128" layer="1"/>
 </signal>
 <signal name="N$7">
